File: esp32cam_shield/esp32cam_shield.kicad_pcb (KiCad board)
At the start: 2 copper layers, 52 parts, among them J1 ESP32 CAM, J2 Battery, J3 Motor, J4 Motor, J5 Motor, J6 Motor, Q1 NMOS, Q2 NMOS, Q3 NMOS, Q4 NMOS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

Commit message: PCB Design DONE.
Parts:
- removed C1: 10u, Capacitor_SMD:C_1206_3216Metric_Pad1.33x1.80mm_HandSolder
- removed C2: 100n, Capacitor_SMD:C_0805_2012Metric_Pad1.18x1.45mm_HandSolder
- removed C3: 10n, Capacitor_SMD:C_0805_2012Metric_Pad1.18x1.45mm_HandSolder
- removed C4, C7: 0.1u, Capacitor_SMD:C_0805_2012Metric_Pad1.18x1.45mm_HandSolder
- removed C5: 1u, Capacitor_SMD:C_0805_2012Metric_Pad1.18x1.45mm_HandSolder
- removed C8: 2.2n, Capacitor_SMD:C_0805_2012Metric_Pad1.18x1.45mm_HandSolder
- removed R1: 4.7k, Resistor_SMD:R_0805_2012Metric_Pad1.20x1.40mm_HandSolder
- removed R2: 3.3k, Resistor_SMD:R_0805_2012Metric_Pad1.20x1.40mm_HandSolder
- removed R3: 3.3K, Resistor_SMD:R_0805_2012Metric_Pad1.20x1.40mm_HandSolder
- removed U1: MPU-6050, Sensor_Motion:InvenSense_QFN-24_4x4mm_P0.5mm
- added J7: Conn_01x08, Connector_PinSocket_2.54mm:PinSocket_1x08_P2.54mm_Vertical, B.Cu at (133.2, 110.0)
- moved R6 82.2 mm to (122.6, 129.1)
- moved C9 81.1 mm to (106.8, 133.8)
- moved C11 80.0 mm to (133.2, 138.5), turned to 90 degrees
- moved J3 78.0 mm to (106.1, 138.5)
- moved Q1 74.8 mm to (107.6, 125.0), turned to 90 degrees
- moved R11 72.8 mm to (142.7, 120.3), turned to 90 degrees
- moved J1 72.2 mm to (114.7, 109.8)
- moved D1 71.2 mm to (113.0, 135.2), turned to 90 degrees
- moved R8 70.1 mm to (118.8, 122.1), turned to 90 degrees
- moved Q3 69.1 mm to (120.3, 134.1), turned to 180 degrees
- moved C12 68.7 mm to (142.0, 127.6), turned to 180 degrees
- moved R4 65.5 mm to (106.2, 117.9), turned to 90 degrees
- moved R9 63.0 mm to (118.8, 117.7), turned to 90 degrees
- moved D3 62.1 mm to (129.2, 137.7), turned to 90 degrees
- moved R5 61.4 mm to (110.2, 117.9), turned to -90 degrees
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Connections:
- Q1 pad 2: /GPIO12 -> /GPIO15
- Q4 pad 2: /GPIO15 -> /GPIO12
- R4 pad 1: /GPIO12 -> /GPIO15
- R7 pad 1: /GPIO15 -> /GPIO12
- R9 pad 2: VCC -> GND
Routing:
- net VCC: track 0.00 -> 157.4 mm
- net +3V3: track 0.00 -> 41.2 mm
- net Net-(D4-A): track 0.00 -> 29.5 mm
- net /GPIO14: track 0.00 -> 22.0 mm
- net GND: track 0.00 -> 16.1 mm, vias 0 -> 2
- net Net-(D1-A): track 0.00 -> 15.4 mm
- net /GPIO12: track 0.00 -> 14.7 mm
- net Net-(D3-A): track 0.00 -> 13.7 mm
- net Net-(U2-SW): track 0.00 -> 13.6 mm
- net Net-(U2-EN): track 0.00 -> 12.3 mm
- net Net-(D2-A): track 0.00 -> 11.4 mm
- net Net-(D7-A): track 0.00 -> 9.75 mm
- net /GPIO15: track 0.00 -> 9.65 mm
- net Net-(U2-FB): track 0.00 -> 9.44 mm
- net /GPIO13: track 0.00 -> 8.25 mm
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- added copper zone on F.Cu, net GND
