File: esp32cam_shield/esp32cam_shield.kicad_sch (KiCad schematic)
At the start: 52 parts, among them J1 ESP32 CAM, J2 Battery, J3 Motor, J4 Motor, J5 Motor, J6 Motor, Q1 NMOS, Q2 NMOS, Q3 NMOS, Q4 NMOS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

Commit message: MPU-6050 modul
Parts:
- removed C1: 10u, Capacitor_SMD:C_1206_3216Metric_Pad1.33x1.80mm_HandSolder, symbol Device:C
- removed C3: 10n, Capacitor_SMD:C_0805_2012Metric_Pad1.18x1.45mm_HandSolder, symbol Device:C
- removed C4, C7: 0.1u, Capacitor_SMD:C_0805_2012Metric_Pad1.18x1.45mm_HandSolder, symbol Device:C
- removed C5: 1u, Capacitor_SMD:C_0805_2012Metric_Pad1.18x1.45mm_HandSolder, symbol Device:C
- removed C8: 2.2n, Capacitor_SMD:C_0805_2012Metric_Pad1.18x1.45mm_HandSolder, symbol Device:C
- removed R1: 4.7k, Resistor_SMD:R_0805_2012Metric_Pad1.20x1.40mm_HandSolder, symbol Device:R
- removed R2: 3.3k, Resistor_SMD:R_0805_2012Metric_Pad1.20x1.40mm_HandSolder, symbol Device:R
- removed R3: 3.3K, Resistor_SMD:R_0805_2012Metric_Pad1.20x1.40mm_HandSolder, symbol Device:R
- removed U1: MPU-6050, Sensor_Motion:InvenSense_QFN-24_4x4mm_P0.5mm, symbol Sensor_Motion:MPU-6050
- added J7: Conn_01x08, Connector_PinSocket_2.54mm:PinSocket_1x08_P2.54mm_Vertical, symbol Connector_Generic:Conn_01x08
Connections:
- net +3V3: now also J7.8 (Pin_8)
- net GND: now also J7.7 (Pin_7)
- net GPIO1: now also J7.6 (Pin_6)
- net GPIO3: now also J7.5 (Pin_5)

Commit message: PCB Design DONE.
Parts:
- removed C2: 100n, Capacitor_SMD:C_0805_2012Metric_Pad1.18x1.45mm_HandSolder, symbol Device:C
- removed J6: Motor, Connector_Hirose:Hirose_DF13-02P-1.25DSA_1x02_P1.25mm_Vertical, symbol Connector_Generic:Conn_02x01
Connections:
- net GND: now also R9.2
- net VCC: no longer R9.2
Changed lines of the file:
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@@
 (kicad_sch (version 20230121) (generator eeschema)
   (paper "A4")
-  (junction (at 189.23 55.88) (diameter 0) (color 0 0 0 0)
-  )
   (junction (at 71.12 144.78) (diameter 0) (color 0 0 0 0)
   )
@@
   (junction (at 83.82 25.4) (diameter 0) (color 0 0 0 0)
   )
-  (junction (at 157.48 138.43) (diameter 0) (color 0 0 0 0)
-  )
   (junction (at 142.24 144.78) (diameter 0) (color 0 0 0 0)
   )
@@
     (stroke (width 0) (type default))
   )
-  (wire (pts (xy 189.23 55.88) (xy 194.31 55.88))
+  (wire (pts (xy 177.8 55.88) (xy 194.31 55.88))
     (stroke (width 0) (type default))
   )
@@
     (stroke (width 0) (type default))
   )
-  (wire (pts (xy 157.48 132.08) (xy 157.48 138.43))
-    (stroke (width 0) (type default))
-  )
   (wire (pts (xy 186.69 86.36) (xy 190.5 86.36))
     (stroke (width 0) (type default))
@@
     (stroke (width 0) (type default))
   )
-  (wire (pts (xy 177.8 55.88) (xy 189.23 55.88))
-    (stroke (width 0) (type default))
-  )
   (wire (pts (xy 218.44 139.7) (xy 229.87 139.7))
     (stroke (width 0) (type default))
@@
     (stroke (width 0) (type default))
   )
-  (wire (pts (xy 133.35 91.44) (xy 133.35 90.17))
+  (wire (pts (xy 133.35 92.71) (xy 133.35 90.17))
     (stroke (width 0) (type default))
   )
@@
     (stroke (width 0) (type default))
   )
-  (wire (pts (xy 135.89 91.44) (xy 133.35 91.44))
+  (wire (pts (xy 135.89 92.71) (xy 133.35 92.71))
     (stroke (width 0) (type default))
   )
@@
     (stroke (width 0) (type default))
   )
-  (wire (pts (xy 144.78 85.09) (xy 132.08 85.09))
-    (stroke (width 0) (type default))
-  )
-  (wire (pts (xy 157.48 144.78) (xy 157.48 138.43))
+  (wire (pts (xy 151.13 85.09) (xy 132.08 85.09))
+    (stroke (width 0) (type default))
+  )
+  (wire (pts (xy 157.48 132.08) (xy 157.48 144.78))
     (stroke (width 0) (type default))
   )
@@
     (effects (font (size 1.27 1.27)) (justify left bottom))
   )
-  (label "GPIO3" (at 135.89 91.44 0) (fields_autoplaced)
+  (label "GPIO3" (at 135.89 92.71 0) (fields_autoplaced)
     (effects (font (size 1.27 1.27)) (justify left bottom))
   )
@@
     )
   )
-  (symbol (lib_id "power:GND") (at 189.23 63.5 0) (unit 1)
-    (in_bom yes) (on_board yes) (dnp no) (fields_autoplaced)
-    (property "Reference" "#PWR04" (at 189.23 69.85 0)
-      (effects (font (size 1.27 1.27)) hide)
-    )
-    (property "Value" "GND" (at 189.23 68.58 0)
-      (effects (font (size 1.27 1.27)))
-    )
-    (property "Footprint" "" (at 189.23 63.5 0)
-      (effects (font (size 1.27 1.27)) hide)
-    )
-    (property "Datasheet" "" (at 189.23 63.5 0)
-      (effects (font (size 1.27 1.27)) hide)
-    )
-    (pin "1")
-    (instances
-      (project "esp32cam_shield"
-        (path "/fdf3d5c5-c89d-4fce-9f43-d1897c15a430"
-          (reference "#PWR04") (unit 1)
-        )
-      )
-    )
-  )
   (symbol (lib_id "Device:R") (at 77.47 162.56 0) (unit 1)
     (in_bom yes) (on_board yes) (dnp no) (fields_autoplaced)
@@
     )
   )
-  (symbol (lib_id "power:GND") (at 144.78 85.09 0) (unit 1)
-    (in_bom yes) (on_board yes) (dnp no) (fields_autoplaced)
-    (property "Reference" "#PWR08" (at 144.78 91.44 0)
-      (effects (font (size 1.27 1.27)) hide)
-    )
-    (property "Value" "GND" (at 144.78 90.17 0)
-      (effects (font (size 1.27 1.27)))
-    )
-    (property "Footprint" "" (at 144.78 85.09 0)
-      (effects (font (size 1.27 1.27)) hide)
-    )
-    (property "Datasheet" "" (at 144.78 85.09 0)
+  (symbol (lib_id "power:GND") (at 151.13 85.09 0) (unit 1)
+    (in_bom yes) (on_board yes) (dnp no) (fields_autoplaced)
+    (property "Reference" "#PWR08" (at 151.13 91.44 0)
+      (effects (font (size 1.27 1.27)) hide)
+    )
+    (property "Value" "GND" (at 151.13 90.17 0)
+      (effects (font (size 1.27 1.27)))
+    )
+    (property "Footprint" "" (at 151.13 85.09 0)
+      (effects (font (size 1.27 1.27)) hide)
+    )
+    (property "Datasheet" "" (at 151.13 85.09 0)
       (effects (font (size 1.27 1.27)) hide)
     )
@@
     )
   )
-  (symbol (lib_id "Device:C") (at 189.23 59.69 0) (unit 1)
-    (in_bom yes) (on_board yes) (dnp no) (fields_autoplaced)
-    (property "Reference" "C2" (at 193.04 59.055 0)
-      (effects (font (size 1.27 1.27)) (justify left))
-    )
-    (property "Value" "100n" (at 193.04 61.595 0)
-      (effects (font (size 1.27 1.27)) (justify left))
-    )
-    (property "Footprint" "Capacitor_SMD:C_0805_2012Metric_Pad1.18x1.45mm_HandSolder" (at 190.1952 63.5 0)
-      (effects (font (size 1.27 1.27)) hide)
-    )
-    (property "Datasheet" "~" (at 189.23 59.69 0)
-      (effects (font (size 1.27 1.27)) hide)
-    )
-    (pin "1")
-    (pin "2")
-    (instances
-      (project "esp32cam_shield"
-        (path "/fdf3d5c5-c89d-4fce-9f43-d1897c15a430"
-          (reference "C2") (unit 1)
-        )
-      )
-    )
-  )
   (symbol (lib_id "power:GND") (at 111.76 167.64 0) (unit 1)
     (in_bom yes) (on_board yes) (dnp no) (fields_autoplaced)
@@
         (path "/fdf3d5c5-c89d-4fce-9f43-d1897c15a430"
           (reference "R9") (unit 1)
+        )
+      )
+    )
+  )
+  (symbol (lib_id "power:GND") (at 229.87 149.86 0) (unit 1)
+    (in_bom yes) (on_board yes) (dnp no) (fields_autoplaced)
+    (property "Reference" "#PWR04" (at 229.87 156.21 0)
+      (effects (font (size 1.27 1.27)) hide)
+    )
+    (property "Value" "GND" (at 229.87 154.94 0)
+      (effects (font (size 1.27 1.27)))
+    )
+    (property "Footprint" "" (at 229.87 149.86 0)
+      (effects (font (size 1.27 1.27)) hide)
+    )
+    (property "Datasheet" "" (at 229.87 149.86 0)
+      (effects (font (size 1.27 1.27)) hide)
+    )
+    (pin "1")
+    (instances
+      (project "esp32cam_shield"
+        (path "/fdf3d5c5-c89d-4fce-9f43-d1897c15a430"
+          (reference "#PWR04") (unit 1)
         )
       )
@@
     )
   )
-  (symbol (lib_id "Connector_Generic:Conn_02x01") (at 162.56 138.43 0) (unit 1)
-    (in_bom yes) (on_board yes) (dnp no) (fields_autoplaced)
-    (property "Reference" "J6" (at 163.83 133.35 0)
-      (effects (font (size 1.27 1.27)))
-    )
-    (property "Value" "Motor" (at 163.83 135.89 0)
-      (effects (font (size 1.27 1.27)))
-    )
-    (property "Footprint" "Connector_Hirose:Hirose_DF13-02P-1.25DSA_1x02_P1.25mm_Vertical" (at 162.56 138.43 0)
-      (effects (font (size 1.27 1.27)) hide)
-    )
-    (property "Datasheet" "~" (at 162.56 138.43 0)
-      (effects (font (size 1.27 1.27)) hide)
-    )
-    (pin "1")
-    (pin "2")
-    (instances
-      (project "esp32cam_shield"
-        (path "/fdf3d5c5-c89d-4fce-9f43-d1897c15a430"
-          (reference "J6") (unit 1)
-        )
-      )
-    )
-  )
   (symbol (lib_id "power:GND") (at 207.01 55.88 0) (unit 1)
     (in_bom yes) (on_board yes) (dnp no) (fields_autoplaced)
@@
         )
       )
-    )
-  )
-  (symbol (lib_id "power:VCC") (at 229.87 149.86 180) (unit 1)
-    (in_bom yes) (on_board yes) (dnp no) (fields_autoplaced)
-    (property "Reference" "#PWR032" (at 229.87 146.05 0)
-      (effects (font (size 1.27 1.27)) hide)
-    )
-    (property "Value" "VBAT" (at 229.87 154.94 0)
-      (effects (font (size 1.27 1.27)))
-    )
-    (property "Footprint" "" (at 229.87 149.86 0)
-      (effects (font (size 1.27 1.27)) hide)
-    )
-    (property "Datasheet" "" (at 229.87 149.86 0)
-      (effects (font (size 1.27 1.27)) hide)
-    )
-    (pin "1")
-    (instances
-      (project "esp32cam_shield"
-        (path "/fdf3d5c5-c89d-4fce-9f43-d1897c15a430"
-          (reference "#PWR032") (unit 1)
-        )
-      )
